Commit message: added red plug

File: assets/factory/urdf/factory_kuka_mod.urdf (robot description, URDF)
Before this commit: robot kuka, 19 links, 18 joints
Links:
- removed link iiwa7_base_link
- removed link iiwa7_link_ee
- added link dummy_ft_link, mass 0.1; collision cylinder length=0.06 radius=0.04; visual cylinder length=0.06 radius=0.04
- added link kuka_fingertip_centered
- link iiwa7_link_0: geometry collision mesh filename=../../urdf/kuka_openhand_description/meshes/iiwa14/collisio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; visual mesh filename=../../urdf/kuka_openhand_description/meshes/iiwa14/visual/l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
- link iiwa7_link_1: mass 3.4525 -> 4; geometry collision mesh filename=../../urdf/kuka_openhand_description/meshes/iiwa14/collisio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; visual mesh filename=../../urdf/kuka_openhand_description/meshes/iiwa14/visual/l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
- link iiwa7_link_2: mass 3.4821 -> 4; geometry collision mesh filename=../../urdf/kuka_openhand_description/meshes/iiwa14/collisio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; visual mesh filename=../../urdf/kuka_openhand_description/meshes/iiwa14/visual/l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
- link iiwa7_link_3: mass 4.05623 -> 3; geometry collision mesh filename=../../urdf/kuka_openhand_description/meshes/iiwa14/collisio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; visual mesh filename=../../urdf/kuka_openhand_description/meshes/iiwa14/visual/l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
- link iiwa7_link_4: mass 3.4822 -> 2.7; geometry collision mesh filename=../../urdf/kuka_openhand_description/meshes/iiwa14/collisio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; visual mesh filename=../../urdf/kuka_openhand_description/meshes/iiwa14/visual/l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
- link iiwa7_link_5: mass 2.1633 -> 1.7; geometry collision mesh filename=../../urdf/kuka_openhand_description/meshes/iiwa14/collisio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; visual mesh filename=../../urdf/kuka_openhand_description/meshes/iiwa14/visual/l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
- link iiwa7_link_6: mass 2.3466 -> 1.8; geometry collision mesh filename=../../urdf/kuka_openhand_description/meshes/iiwa14/collisio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; visual mesh filename=../../urdf/kuka_openhand_description/meshes/iiwa14/visual/l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
- link iiwa7_link_7: mass 3.129 -> 0.3; geometry collision mesh filename=../../urdf/kuka_openhand_description/meshes/iiwa14/collisio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; visual mesh filename=../../urdf/kuka_openhand_description/meshes/iiwa14/visual/l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
Joints:
- removed joint iiwa7_base_link_iiwa7_joint
- added joint iiwa_ft_base_joint: type fixed, parent iiwa7_link_7, child dummy_ft_link, origin xyz=0 0 0.075 rpy=0 0 0
- joint iiwa7_joint_1: limit lower=-2.96705972839 upper=2.96705972839 effort=300 velocity=10 -> lower=-2.96705972839 upper=2.96705972839 effort=300 velocity=2; origin xyz=0 0 0.15 rpy=0 0 0 -> xyz=0 0 0.1575 rpy=0 0 0
- joint iiwa7_joint_2: limit lower=-2.09439510239 upper=2.09439510239 effort=300 velocity=10 -> lower=-2.09439510239 upper=2.09439510239 effort=300 velocity=2; origin xyz=0 0 0.19 rpy=1.57079632679   0 3.14159265359 -> xyz=0 0 0.2025 rpy=1.57079632679   0 3.14159265359
- joint iiwa7_joint_3: limit lower=-2.96705972839 upper=2.96705972839 effort=300 velocity=10 -> lower=-2.96705972839 upper=2.96705972839 effort=300 velocity=2; origin xyz=0 0.21 0 rpy=1.57079632679 0 3.14159265359 -> xyz=0 0.2045 0 rpy=1.57079632679 0 3.14159265359
- joint iiwa7_joint_4: limit lower=-2.09439510239 upper=2.09439510239 effort=300 velocity=10 -> lower=-2.09439510239 upper=2.09439510239 effort=300 velocity=2; origin xyz=0 0 0.19 rpy=1.57079632679 0 0 -> xyz=0 0 0.2155 rpy=1.57079632679 0 0
- joint iiwa7_joint_5: limit lower=-2.96705972839 upper=2.96705972839 effort=300 velocity=10 -> lower=-2.96705972839 upper=2.96705972839 effort=300 velocity=2; origin xyz=0 0.21 0 rpy=-1.57079632679 3.14159265359 0 -> xyz=0 0.1845 0 rpy=-1.57079632679 3.14159265359 0
- joint iiwa7_joint_6: limit lower=-2.09439510239 upper=2.09439510239 effort=300 velocity=10 -> lower=-2.09439510239 upper=2.09439510239 effort=300 velocity=2; origin xyz=0 0.06070 0.19 rpy=1.57079632679 0 0 -> xyz=0 0 0.2155 rpy=1.57079632679 0 0
- joint iiwa7_joint_7: limit lower=-3.05432619099 upper=3.05432619099 effort=300 velocity=10 -> lower=-3.05432619099 upper=3.05432619099 effort=300 velocity=2; origin xyz=0 0.081 0.06070 rpy=-1.57079632679 3.14159265359 0 -> xyz=0 0.081 0 rpy=-1.57079632679 3.14159265359 0
- joint iiwa7_joint_ee: child iiwa7_link_ee -> kuka_fingertip_centered; origin xyz=0 0 0.071 rpy=0 0 0 -> xyz=-0.12 -0.01 -0.000 rpy=0 -1.57079632679 0; parent iiwa7_link_7 -> gripper_base_link
- joint iiwa_gripper_base_joint: origin xyz=0 0 0.1 rpy=0 1.57079632679 0 -> xyz=0 0 0.09 rpy=0 1.57079632679 0; parent iiwa7_link_7 -> dummy_ft_link

File: assets/factory/urdf/red_round_peg_15in.urdf (robot description, URDF)
Before this commit: robot factory_round_peg_16mm_loose, 1 links, 0 joints
Links:
- link factory_round_peg_16mm_loose: geometry collision mesh filename=../mesh/factory_insertion/red_round_peg_15in.obj; visual mesh filename=../mesh/factory_insertion/red_round_peg_15in.obj
