Commit message: changed substep to 5

File: assets/factory/urdf/green_round_hole_1_5in.urdf (robot description, URDF)
Before this commit: robot round_hole_1_5in_sim_loose, 1 links, 0 joints
Links:
- removed link round_hole_1_5in_sim_loose
- added link green_round_hole_1_5in; collision mesh filename=../mesh/factory_insertion/green_round_hole_1_5in.obj; visual mesh filename=../mesh/factory_insertion/green_round_hole_1_5in.obj

File: assets/factory/urdf/red_round_peg_1_5in.urdf (robot description, URDF)
Before this commit: robot red_round_peg_15in, 1 links, 0 joints
Links:
- link red_round_peg_15in: geometry collision mesh filename=../mesh/factory_insertion/red_round_peg_1_5in.obj; visual mesh filename=../mesh/factory_insertion/red_round_peg_1_5in.obj

File: assets/factory/urdf/red_triangle_hole.urdf (robot description, URDF)
Before this commit: robot red_triangle_hole, 1 links, 0 joints
Links:
- link red_triangle_hole: geometry collision mesh filename=../mesh/factory_insertion/red_triangle_hole.obj; visual mesh filename=../mesh/factory_insertion/red_triangle_hole.obj
