Commit message: useless commit

File: assets/factory/urdf/green_round_hole_2in.urdf (robot description, URDF)
Before this commit: robot factory_round_peg_16mm_loose, 1 links, 0 joints
Links:
- removed link factory_round_peg_16mm_loose
- added link green_round_peg_16mm_loose; collision mesh filename=../mesh/factory_insertion/2inNewShamrockBox.obj; visual mesh filename=../mesh/factory_insertion/2inNewShamrockBox.obj

File: assets/factory/urdf/yellow_round_peg_2in.urdf (robot description, URDF)
Before this commit: robot factory_round_peg_16mm_loose, 1 links, 0 joints
Links:
- removed link factory_round_peg_16mm_loose
- added link yellow_round_peg_16mm_loose; collision mesh filename=../mesh/factory_insertion/yellow_round_peg_2in.obj; visual mesh filename=../mesh/factory_insertion/yellow_round_peg_2in.obj

Commit message: added new object, resized holes

File: assets/factory/urdf/green_round_hole_2in.urdf (robot description, URDF)
Before this commit: robot green_round_peg_16mm_loose, 1 links, 0 joints
Links:
- removed link green_round_peg_16mm_loose
- added link round_hole_2in_sim_loose; collision mesh filename=../mesh/factory_insertion/round_hole_2in_sim_loose.obj scale=0.00100 0.00100 0.00100; visual mesh filename=../mesh/factory_insertion/round_hole_2in_sim_loose.obj scale=0.00100 0.00100 0.00100

File: assets/factory/urdf/red_round_peg_15in.urdf (robot description, URDF)
Before this commit: robot factory_round_peg_16mm_loose, 1 links, 0 joints
Links:
- removed link factory_round_peg_16mm_loose
- added link red_round_peg_15in; collision mesh filename=../mesh/factory_insertion/red_round_peg_15in.obj; visual mesh filename=../mesh/factory_insertion/red_round_peg_15in.obj

File: assets/factory/urdf/yellow_round_peg_2in.urdf (robot description, URDF)
Before this commit: robot yellow_round_peg_16mm_loose, 1 links, 0 joints
Links:
- removed link yellow_round_peg_16mm_loose
- added link yellow_round_peg_2in; collision mesh filename=../mesh/factory_insertion/yellow_round_peg_2in.obj; visual mesh filename=../mesh/factory_insertion/yellow_round_peg_2in.obj

Commit message: test old hole

File: assets/factory/urdf/green_round_hole_2in.urdf (robot description, URDF)
Before this commit: robot round_hole_2in_sim_loose, 1 links, 0 joints
Links:
- link round_hole_2in_sim_loose: geometry collision mesh filename=../mesh/factory_insertion/round_hole_2in_sim_loose.obj scale=0.00100 0.00100 0.00100; visual mesh filename=../mesh/factory_insertion/round_hole_2in_sim_loose.obj scale=0.00100 0.00100 0.00100

Commit message: with datasets

File: assets/factory/urdf/green_round_hole_2in.urdf (robot description, URDF)
Before this commit: robot round_hole_2in_sim_loose, 1 links, 0 joints
Links:
- link round_hole_2in_sim_loose: geometry collision mesh filename=../mesh/factory_insertion/socket.obj; visual mesh filename=../mesh/factory_insertion/socket.obj

Commit message: with memory leak

File: assets/factory/urdf/green_round_hole_2in.urdf (robot description, URDF)
Before this commit: robot round_hole_2in_sim_loose, 1 links, 0 joints
Links:
- link round_hole_2in_sim_loose: geometry collision mesh filename=../mesh/factory_insertion/green_round_hole_2in.obj; visual mesh filename=../mesh/factory_insertion/green_round_hole_2in.obj
