Commit message: rotate

File: assets/factory/urdf/factory_rectangular_hole_32mm.urdf (robot description, URDF)
Before this commit: robot factory_rectangular_hole_16mm, 1 links, 0 joints
Links:
- link factory_rectangular_hole_16mm: geometry collision mesh filename=../mesh/factory_insertion/factory_rectangular_hole_32mm_sub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; visual mesh filename=../mesh/factory_insertion/factory_rectangular_hole_32mm_sub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

File: assets/factory/urdf/factory_square_hole_32mm.urdf (robot description, URDF)
Before this commit: robot factory_rectangular_hole_16mm, 1 links, 0 joints
Links:
- link factory_rectangular_hole_16mm: geometry collision mesh filename=../mesh/factory_insertion/factory_square_hole_32mm_subdiv_3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; visual mesh filename=../mesh/factory_insertion/factory_square_hole_32mm_subdiv_3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
