Commit message: approx center app

File: assets/factory/urdf/factory_kuka.urdf (robot description, URDF)
Before this commit: robot kuka, 18 links, 17 joints
Joints:
- joint iiwa7_joint_ee: origin xyz=0 0 0.071 rpy=0 0 0 -> xyz=-0.12 -0.01 -0.000 rpy=0 -1.57079632679 0

Commit message: changed to iiwa14 + dummy ft

File: assets/factory/urdf/factory_kuka.urdf (robot description, URDF)
Before this commit: robot kuka, 18 links, 17 joints
Links:
- added link dummy_ft_link, mass 0.1; collision cylinder length=0.06 radius=0.04; visual cylinder length=0.06 radius=0.04
- link iiwa7_link_0: geometry collision mesh filename=../../urdf/kuka_openhand_description/meshes/iiwa14/collisio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; visual mesh filename=../../urdf/kuka_openhand_description/meshes/iiwa14/visual/l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
- link iiwa7_link_1: mass 3.4525 -> 4; geometry collision mesh filename=../../urdf/kuka_openhand_description/meshes/iiwa14/collisio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; visual mesh filename=../../urdf/kuka_openhand_description/meshes/iiwa14/visual/l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
- link iiwa7_link_2: mass 3.4821 -> 4; geometry collision mesh filename=../../urdf/kuka_openhand_description/meshes/iiwa14/collisio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; visual mesh filename=../../urdf/kuka_openhand_description/meshes/iiwa14/visual/l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
- link iiwa7_link_3: mass 4.05623 -> 3; geometry collision mesh filename=../../urdf/kuka_openhand_description/meshes/iiwa14/collisio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; visual mesh filename=../../urdf/kuka_openhand_description/meshes/iiwa14/visual/l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
- link iiwa7_link_4: mass 3.4822 -> 2.7; geometry collision mesh filename=../../urdf/kuka_openhand_description/meshes/iiwa14/collisio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; visual mesh filename=../../urdf/kuka_openhand_description/meshes/iiwa14/visual/l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
- link iiwa7_link_5: mass 2.1633 -> 1.7; geometry collision mesh filename=../../urdf/kuka_openhand_description/meshes/iiwa14/collisio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; visual mesh filename=../../urdf/kuka_openhand_description/meshes/iiwa14/visual/l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
- link iiwa7_link_6: mass 2.3466 -> 1.8; geometry collision mesh filename=../../urdf/kuka_openhand_description/meshes/iiwa14/collisio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; visual mesh filename=../../urdf/kuka_openhand_description/meshes/iiwa14/visual/l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
- link iiwa7_link_7: mass 3.129 -> 0.3; geometry collision mesh filename=../../urdf/kuka_openhand_description/meshes/iiwa14/collisio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; visual mesh filename=../../urdf/kuka_openhand_description/meshes/iiwa14/visual/l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
Joints:
- added joint iiwa_ft_base_joint: type fixed, parent iiwa7_link_7, child dummy_ft_link, origin xyz=0 0 0.075 rpy=0 0 0
- joint iiwa7_joint_1: limit lower=-2.96705972839 upper=2.96705972839 effort=300 velocity=10 -> lower=-2.96705972839 upper=2.96705972839 effort=300 velocity=2; origin xyz=0 0 0.15 rpy=0 0 0 -> xyz=0 0 0.1575 rpy=0 0 0
- joint iiwa7_joint_2: limit lower=-2.09439510239 upper=2.09439510239 effort=300 velocity=10 -> lower=-2.09439510239 upper=2.09439510239 effort=300 velocity=2; origin xyz=0 0 0.19 rpy=1.57079632679   0 3.14159265359 -> xyz=0 0 0.2025 rpy=1.57079632679   0 3.14159265359
- joint iiwa7_joint_3: limit lower=-2.96705972839 upper=2.96705972839 effort=300 velocity=10 -> lower=-2.96705972839 upper=2.96705972839 effort=300 velocity=2; origin xyz=0 0.21 0 rpy=1.57079632679 0 3.14159265359 -> xyz=0 0.2045 0 rpy=1.57079632679 0 3.14159265359
- joint iiwa7_joint_4: limit lower=-2.09439510239 upper=2.09439510239 effort=300 velocity=10 -> lower=-2.09439510239 upper=2.09439510239 effort=300 velocity=2; origin xyz=0 0 0.19 rpy=1.57079632679 0 0 -> xyz=0 0 0.2155 rpy=1.57079632679 0 0
- joint iiwa7_joint_5: limit lower=-2.96705972839 upper=2.96705972839 effort=300 velocity=10 -> lower=-2.96705972839 upper=2.96705972839 effort=300 velocity=2; origin xyz=0 0.21 0 rpy=-1.57079632679 3.14159265359 0 -> xyz=0 0.1845 0 rpy=-1.57079632679 3.14159265359 0
- joint iiwa7_joint_6: limit lower=-2.09439510239 upper=2.09439510239 effort=300 velocity=10 -> lower=-2.09439510239 upper=2.09439510239 effort=300 velocity=2; origin xyz=0 0.06070 0.19 rpy=1.57079632679 0 0 -> xyz=0 0 0.2155 rpy=1.57079632679 0 0
- joint iiwa7_joint_7: limit lower=-3.05432619099 upper=3.05432619099 effort=300 velocity=10 -> lower=-3.05432619099 upper=3.05432619099 effort=300 velocity=2; origin xyz=0 0.081 0.06070 rpy=-1.57079632679 3.14159265359 0 -> xyz=0 0.081 0 rpy=-1.57079632679 3.14159265359 0
- joint iiwa_gripper_base_joint: origin xyz=0 0 0.1 rpy=0 1.57079632679 0 -> xyz=0 0 0.09 rpy=0 1.57079632679 0; parent iiwa7_link_7 -> dummy_ft_link

Commit message: sdf fix?

File: assets/factory/urdf/factory_kuka.urdf (robot description, URDF)
Before this commit: robot kuka, 19 links, 18 joints
Links:
- link finger_1_3: geometry collision cylinder length=0.028 radius=0.012; visual mesh filename=../../urdf/kuka_openhand_description/meshes/allsight/allsig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
- link finger_2_3: geometry collision cylinder length=0.028 radius=0.012; visual mesh filename=../../urdf/kuka_openhand_description/meshes/allsight/allsig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
- link finger_3_3: geometry collision cylinder length=0.028 radius=0.012; visual mesh filename=../../urdf/kuka_openhand_description/meshes/allsight/allsig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

Commit message: removed sdf from object

File: assets/factory/urdf/factory_kuka.urdf (robot description, URDF)
Before this commit: robot kuka, 19 links, 18 joints
Links:
- link finger_1_3: geometry collision mesh filename=../../urdf/kuka_openhand_description/meshes/allsight/allsig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; visual mesh filename=../../urdf/kuka_openhand_description/meshes/allsight/allsig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
- link finger_2_3: geometry collision mesh filename=../../urdf/kuka_openhand_description/meshes/allsight/allsig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; visual mesh filename=../../urdf/kuka_openhand_description/meshes/allsight/allsig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
- link finger_3_3: geometry collision mesh filename=../../urdf/kuka_openhand_description/meshes/allsight/allsig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; visual mesh filename=../../urdf/kuka_openhand_description/meshes/allsight/allsig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
Joints:
- joint base_to_finger_1_1: limit lower=0 upper=1.57079632679 effort=100 velocity=2 -> lower=0 upper=1.57079632679 effort=2 velocity=2
- joint base_to_finger_2_1: limit lower=-1.57079632679 upper=0 effort=100 velocity=2 -> lower=-1.57079632679 upper=0 effort=2 velocity=2
- joint base_to_finger_3_2: limit lower=-0.1 upper=3.0 effort=100 velocity=2 -> lower=-0.1 upper=3.0 effort=2 velocity=2
- joint finger_1_1_to_finger_1_2: limit lower=-0.1 upper=3.0 effort=100 velocity=2 -> lower=-0.1 upper=3.0 effort=2 velocity=2
- joint finger_1_2_to_finger_1_3: limit lower=0.0 upper=1.27 effort=100 velocity=2 -> lower=0.0 upper=1.27 effort=2 velocity=2
- joint finger_2_1_to_finger_2_2: limit lower=-0.1 upper=3.0 effort=100 velocity=2 -> lower=-0.1 upper=3.0 effort=2 velocity=2
- joint finger_2_2_to_finger_2_3: limit lower=0.0 upper=1.27 effort=100 velocity=2 -> lower=0.0 upper=1.27 effort=2 velocity=2
- joint finger_3_2_to_finger_3_3: limit lower=0.0 upper=1.27 effort=100 velocity=2 -> lower=0.0 upper=1.27 effort=2 velocity=2

Commit message: urdf change

File: assets/factory/urdf/factory_kuka.urdf (robot description, URDF)
Before this commit: robot kuka, 19 links, 18 joints
Links:
- added link mount_1_3, mass 0.05; collision mesh filename=../../urdf/kuka_openhand_description/meshes/allsight/allsig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; visual mesh filename=../../urdf/kuka_openhand_description/meshes/allsight/allsig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
- added link mount_2_3, mass 0.05; collision mesh filename=../../urdf/kuka_openhand_description/meshes/allsight/allsig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; visual mesh filename=../../urdf/kuka_openhand_description/meshes/allsight/allsig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
- added link mount_3_3, mass 0.05; collision mesh filename=../../urdf/kuka_openhand_description/meshes/allsight/allsig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; visual mesh filename=../../urdf/kuka_openhand_description/meshes/allsight/allsig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
- link dummy_ft_link: geometry collision cylinder length=0.08 radius=0.04; visual cylinder length=0.08 radius=0.04
- link finger_1_1: mass 0.1 -> 0.05
- link finger_1_2: mass 0.1 -> 0.05
- link finger_1_3: mass 0.1 -> 0.05
- link finger_2_1: mass 0.1 -> 0.05
- link finger_2_2: mass 0.1 -> 0.05
- link finger_2_3: mass 0.1 -> 0.05
- link finger_3_2: mass 0.1 -> 0.05
- link finger_3_3: mass 0.1 -> 0.05
- link iiwa7_link_7: geometry collision mesh filename=../../urdf/kuka_openhand_description/meshes/iiwa14/visual/l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; visual mesh filename=../../urdf/kuka_openhand_description/meshes/iiwa14/visual/l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
Joints:
- added joint finger_1_2_to_finger_1_3_tip: type fixed, parent mount_1_3, child finger_1_3, origin xyz=0.025 0.003 0 rpy=1.57079632679 0 0
- added joint finger_2_2_to_finger_2_3_tip: type fixed, parent mount_2_3, child finger_2_3, origin xyz=0.025 0.003 0 rpy=1.57079632679 0 0
- added joint finger_3_2_to_finger_3_3_tip: type fixed, parent mount_3_3, child finger_3_3, origin xyz=0.025 0.003 0 rpy=1.57079632679 0 0
- joint base_to_finger_1_1: limit lower=0 upper=1.57079632679 effort=2 velocity=2 -> lower=0 upper=1.57079632679 effort=3 velocity=2
- joint base_to_finger_2_1: limit lower=-1.57079632679 upper=0 effort=2 velocity=2 -> lower=-1.57079632679 upper=0 effort=3 velocity=2
- joint base_to_finger_3_2: limit lower=-0.1 upper=3.0 effort=2 velocity=2 -> lower=-0.1 upper=3.0 effort=3 velocity=2; origin xyz=-0.023 0.045 0.000000 rpy=0 0 0 -> xyz=-0.023 0.047 0.000000 rpy=0 0 0
- joint finger_1_1_to_finger_1_2: limit lower=-0.1 upper=3.0 effort=2 velocity=2 -> lower=-0.1 upper=3.0 effort=3 velocity=2; origin xyz=-0.02 0.00725 0 rpy=0 0 0 -> xyz=-0.023 0.00725 0 rpy=0 0 0
- joint finger_1_2_to_finger_1_3: axis 0 1 0 -> 0 0 1; child finger_1_3 -> mount_1_3; limit lower=0.0 upper=1.27 effort=2 velocity=2 -> lower=0.0 upper=1.27 effort=3 velocity=2; origin xyz=0.000800 0.072 0 rpy=1.57079632679 0 1.57079632679 -> xyz=0.0008 0.063 0 rpy=0 0 1.57079632679
- joint finger_2_1_to_finger_2_2: limit lower=-0.1 upper=3.0 effort=2 velocity=2 -> lower=-0.1 upper=3.0 effort=3 velocity=2
- joint finger_2_2_to_finger_2_3: axis 0 1 0 -> 0 0 1; child finger_2_3 -> mount_2_3; limit lower=0.0 upper=1.27 effort=2 velocity=2 -> lower=0.0 upper=1.27 effort=3 velocity=2; origin xyz=0.000800 0.072 0 rpy=1.57079632679 0 1.57079632679 -> xyz=0.0008 0.063 0 rpy=0 0 1.57079632679
- joint finger_3_2_to_finger_3_3: axis 0 1 0 -> 0 0 1; child finger_3_3 -> mount_3_3; limit lower=0.0 upper=1.27 effort=2 velocity=2 -> lower=0.0 upper=1.27 effort=3 velocity=2; origin xyz=0.000800 0.072 0 rpy=1.57079632679 0 1.57079632679 -> xyz=0.0008 0.063 0 rpy=0 0 1.57079632679
- joint iiwa7_joint_ee: origin xyz=0.00 -0.01 0.21 rpy=0 0 0 -> xyz=0.00 -0.01 0.23 rpy=0 0 0
- joint iiwa_ft_base_joint: origin xyz=0 0 0.075 rpy=0 0 0 -> xyz=0 0 0.11 rpy=0 0 0
- joint iiwa_gripper_base_joint: origin xyz=0 0 0.09 rpy=0 1.57079632679 0 -> xyz=0 0 0.21 rpy=0 1.57079632679 0; parent dummy_ft_link -> iiwa7_link_7

Commit message: push with slower vel in urdf

File: assets/factory/urdf/factory_kuka.urdf (robot description, URDF)
Before this commit: robot kuka, 22 links, 21 joints
Joints:
- joint iiwa7_joint_1: limit lower=-2.96705972839 upper=2.96705972839 effort=300 velocity=2 -> lower=-2.96705972839 upper=2.96705972839 effort=300 velocity=0.01
- joint iiwa7_joint_2: limit lower=-2.09439510239 upper=2.09439510239 effort=300 velocity=2 -> lower=-2.09439510239 upper=2.09439510239 effort=300 velocity=0.01
- joint iiwa7_joint_3: limit lower=-2.96705972839 upper=2.96705972839 effort=300 velocity=2 -> lower=-2.96705972839 upper=2.96705972839 effort=300 velocity=0.01
- joint iiwa7_joint_4: limit lower=-2.09439510239 upper=2.09439510239 effort=300 velocity=2 -> lower=-2.09439510239 upper=2.09439510239 effort=300 velocity=0.01
- joint iiwa7_joint_5: limit lower=-2.96705972839 upper=2.96705972839 effort=300 velocity=2 -> lower=-2.96705972839 upper=2.96705972839 effort=300 velocity=0.01
- joint iiwa7_joint_6: limit lower=-2.09439510239 upper=2.09439510239 effort=300 velocity=2 -> lower=-2.09439510239 upper=2.09439510239 effort=300 velocity=0.01
- joint iiwa7_joint_7: limit lower=-3.05432619099 upper=3.05432619099 effort=300 velocity=2 -> lower=-3.05432619099 upper=3.05432619099 effort=300 velocity=0.01

Commit message: working in real version

File: assets/factory/urdf/factory_kuka.urdf (robot description, URDF)
Before this commit: robot kuka, 22 links, 21 joints
Joints:
- joint iiwa7_joint_1: limit lower=-2.96705972839 upper=2.96705972839 effort=300 velocity=0.01 -> lower=-2.96705972839 upper=2.96705972839 effort=300 velocity=0.1
- joint iiwa7_joint_2: limit lower=-2.09439510239 upper=2.09439510239 effort=300 velocity=0.01 -> lower=-2.09439510239 upper=2.09439510239 effort=300 velocity=0.1
- joint iiwa7_joint_3: limit lower=-2.96705972839 upper=2.96705972839 effort=300 velocity=0.01 -> lower=-2.96705972839 upper=2.96705972839 effort=300 velocity=0.1
- joint iiwa7_joint_4: limit lower=-2.09439510239 upper=2.09439510239 effort=300 velocity=0.01 -> lower=-2.09439510239 upper=2.09439510239 effort=300 velocity=0.1
- joint iiwa7_joint_5: limit lower=-2.96705972839 upper=2.96705972839 effort=300 velocity=0.01 -> lower=-2.96705972839 upper=2.96705972839 effort=300 velocity=0.1
- joint iiwa7_joint_6: limit lower=-2.09439510239 upper=2.09439510239 effort=300 velocity=0.01 -> lower=-2.09439510239 upper=2.09439510239 effort=300 velocity=0.1
- joint iiwa7_joint_7: limit lower=-3.05432619099 upper=3.05432619099 effort=300 velocity=0.01 -> lower=-3.05432619099 upper=3.05432619099 effort=300 velocity=0.1

Commit message: first update

File: assets/factory/urdf/factory_kuka.urdf (robot description, URDF)
Before this commit: robot kuka, 22 links, 21 joints
Joints:
- joint base_to_finger_1_1: axis 1 0 0 -> (none); limit lower=0 upper=1.57079632679 effort=3 velocity=2 -> (none); origin xyz=-0.003 -0.034 -0.027 rpy=3.14159265359 0 0 -> xyz=-0.003 -0.034 -0.027 rpy=3.84159265359 0 0; type revolute -> fixed
- joint base_to_finger_2_1: axis 1 0 0 -> (none); limit lower=-1.57079632679 upper=0 effort=3 velocity=2 -> (none); origin xyz=-0.003 -0.034 0.027 rpy=3.14159265359 0 0 -> xyz=-0.003 -0.034 0.027 rpy=2.44159265359 0 0; type revolute -> fixed
- joint iiwa7_joint_1: limit lower=-2.96705972839 upper=2.96705972839 effort=300 velocity=2 -> lower=-2.96705972839 upper=2.96705972839 effort=87 velocity=2
- joint iiwa7_joint_2: limit lower=-2.09439510239 upper=2.09439510239 effort=300 velocity=2 -> lower=-2.09439510239 upper=2.09439510239 effort=87 velocity=2
- joint iiwa7_joint_3: limit lower=-2.96705972839 upper=2.96705972839 effort=300 velocity=2 -> lower=-2.96705972839 upper=2.96705972839 effort=87 velocity=2
- joint iiwa7_joint_4: limit lower=-2.09439510239 upper=2.09439510239 effort=300 velocity=2 -> lower=-2.09439510239 upper=2.09439510239 effort=87 velocity=2
- joint iiwa7_joint_5: limit lower=-2.96705972839 upper=2.96705972839 effort=300 velocity=2 -> lower=-2.96705972839 upper=2.96705972839 effort=12 velocity=2
- joint iiwa7_joint_6: limit lower=-2.09439510239 upper=2.09439510239 effort=300 velocity=2 -> lower=-2.09439510239 upper=2.09439510239 effort=12 velocity=2
- joint iiwa7_joint_7: limit lower=-3.05432619099 upper=3.05432619099 effort=300 velocity=2 -> lower=-3.05432619099 upper=3.05432619099 effort=12 velocity=2

Commit message: first push

File: assets/factory/urdf/factory_kuka.urdf (robot description, URDF)
Before this commit: robot kuka, 22 links, 21 joints
Links:
- removed link finger_3_2
- removed link finger_3_3
- removed link mount_3_3
Joints:
- removed joint base_to_finger_3_2
- removed joint finger_3_2_to_finger_3_3
- removed joint finger_3_2_to_finger_3_3_tip
- joint iiwa7_joint_ee: origin xyz=0.00 -0.01 0.23 rpy=0 0 0 -> xyz=0.00 -0.035 0.23 rpy=0 0 0

Commit message: Update

File: assets/factory/urdf/factory_kuka.urdf (robot description, URDF)
Before this commit: robot kuka, 22 links, 21 joints
Links:
- link dummy_ft_link: mass 0.1 -> 0.3
- link gripper_base_link: mass 0.7 -> 0.3
Joints:
- joint base_to_finger_1_1: limit lower=0 upper=1.57079632679 effort=3 velocity=2 -> lower=0 upper=1.57079632679 effort=0.1 velocity=2
- joint base_to_finger_2_1: limit lower=-1.57079632679 upper=0 effort=3 velocity=2 -> lower=-1.57079632679 upper=0 effort=0.1 velocity=2
- joint base_to_finger_3_2: limit lower=-0.1 upper=3.0 effort=3 velocity=2 -> lower=-0.1 upper=3.0 effort=0.1 velocity=2
- joint finger_1_1_to_finger_1_2: limit lower=-0.1 upper=3.0 effort=3 velocity=2 -> lower=-0.1 upper=3.0 effort=0.1 velocity=2
- joint finger_1_2_to_finger_1_3: limit lower=0.0 upper=1.27 effort=3 velocity=2 -> lower=0.0 upper=1.27 effort=0.1 velocity=2
- joint finger_2_1_to_finger_2_2: limit lower=-0.1 upper=3.0 effort=3 velocity=2 -> lower=-0.1 upper=3.0 effort=0.1 velocity=2
- joint finger_2_2_to_finger_2_3: limit lower=0.0 upper=1.27 effort=3 velocity=2 -> lower=0.0 upper=1.27 effort=0.1 velocity=2
- joint finger_3_2_to_finger_3_3: limit lower=0.0 upper=1.27 effort=3 velocity=2 -> lower=0.0 upper=1.27 effort=0.1 velocity=2
